Commit message: merge and update d435

File: urdf/realsense-D435.macro.xacro (robot description, xacro)
@@ -17,5 +17,5 @@
             <origin rpy="0 0 0" xyz="0 0 0"/>
             <geometry>
-                <mesh filename="package://realsense_gazebo_plugin/models/realsense_camera/meshes/realsense.dae"/>
+                <mesh filename="package://realsense_gazebo_plugin/models/realsense_camera/meshes/realsense_d435.stl"/>
             </geometry>
         </visual>
