Commit message: update all namings and briefly reorganize the code

File: urdf/d435_simulation.xacro (robot description, xacro)
@@ -4,11 +4,11 @@
     This is an example of how to use the realsense-rs200 macro function.
 -->
-<robot name="robot_with_D435" xmlns:xacro="http://ros.org/wiki/xacro">
+<robot name="robot_with_d435" xmlns:xacro="http://ros.org/wiki/xacro">
     <link name="world"/>
     <!-- Import macro for realsense-RS200 camera-->
-    <xacro:include filename="$(find realsense_gazebo_plugin)/urdf/realsense-D435.macro.xacro"/>
+    <xacro:include filename="$(find realsense_gazebo_plugin)/urdf/realsense-d435.macro.xacro"/>
     <!-- Create camera instance -->
-    <xacro:realsense-D435 prefix="" parent="world">
+    <xacro:realsense-d435 prefix="" parent="world">
         <origin xyz="0 0 1.0" rpy="0 0 0" />
-    </xacro:realsense-D435>
+    </xacro:realsense-d435>
 </robot>

File: urdf/multi_r200_simulation.xacro (robot description, xacro)
@@ -1,7 +1,7 @@
 <?xml version="1.0"?>
-<robot name="robot_with_two_rs200" xmlns:xacro="http://ros.org/wiki/xacro">
+<robot name="robot_with_two_r200" xmlns:xacro="http://ros.org/wiki/xacro">
     <link name="world"/>
     <!-- Import macro for realsense-RS200 camera-->
-    <xacro:include filename="$(find realsense_gazebo_plugin)/urdf/realsense-RS200.macro.xacro"/>
+    <xacro:include filename="$(find realsense_gazebo_plugin)/urdf/realsense-r200.macro.xacro"/>
     <!-- Create two camera instances -->
     <xacro:realsense-rs200 prefix="left_" parent="world">

File: urdf/r200_simulation.xacro (robot description, xacro)
@@ -4,11 +4,11 @@
     This is an example of how to use the realsense-rs200 macro function.
 -->
-<robot name="robot_with_rs200" xmlns:xacro="http://ros.org/wiki/xacro">
+<robot name="robot_with_r200" xmlns:xacro="http://ros.org/wiki/xacro">
     <link name="world"/>
     <!-- Import macro for realsense-RS200 camera-->
-    <xacro:include filename="$(find realsense_gazebo_plugin)/urdf/realsense-RS200.macro.xacro"/>
+    <xacro:include filename="$(find realsense_gazebo_plugin)/urdf/realsense-r200.macro.xacro"/>
     <!-- Create camera instance -->
-    <xacro:realsense-rs200 prefix="" parent="world">
+    <xacro:realsense-r200 prefix="" parent="world">
         <origin xyz="0 0 1.0" rpy="0 0 0" />
-    </xacro:realsense-rs200>
+    </xacro:realsense-r200>
 </robot>

File: urdf/realsense-d435.macro.xacro (robot description, xacro)
@@ -11,9 +11,9 @@
 -->
 <robot xmlns:xacro="http://ros.org/wiki/xacro">
-<xacro:macro name="realsense-D435" params="prefix parent *origin">
+<xacro:macro name="realsense-d435" params="prefix parent *origin">
     <!-- Camera link -->
-    <link name="${prefix}D435_camera">
+    <link name="${prefix}d435_camera">
         <visual>
-            <origin rpy="0 0 0" xyz="0 0 0"/>
+            <origin rpy="1.57 0 1.57" xyz="0 0 0"/>
             <geometry>
                 <mesh filename="package://realsense_gazebo_plugin/models/realsense_camera/meshes/realsense_d435.stl"/>
@@ -40,5 +40,5 @@
     <joint name="${prefix}realsense_joint" type="fixed">
         <parent link="${parent}"/>
-        <child link="${prefix}D435_camera"/>
+        <child link="${prefix}d435_camera"/>
         <xacro:insert_block name="origin"/>
     </joint>
@@ -50,5 +50,5 @@
     <!-- Joints positioning the virtual links with respect to the camera main link-->
     <joint name="${prefix}color_joint" type="fixed">
-        <parent link="${prefix}D435_camera" />
+        <parent link="${prefix}d435_camera" />
         <child link="${prefix}color" />
         <!-- <origin xyz="0 -0.046 0.004" rpy="0 0 0"/> -->
@@ -57,15 +57,15 @@
     </joint>
     <joint name="${prefix}depth_joint" type="fixed">
-        <parent link="${prefix}D435_camera" />
+        <parent link="${prefix}d435_camera" />
         <child link="${prefix}depth" />
         <origin xyz="0 -0.03 0.004" rpy="0 0 0"/>
     </joint>
     <joint name="${prefix}ired1_joint" type="fixed">
-        <parent link="${prefix}D435_camera" />
+        <parent link="${prefix}d435_camera" />
         <child link="${prefix}ired1" />
         <origin xyz="0 -0.06 0.004" rpy="0 0 0"/>
     </joint>
     <joint name="${prefix}ired2_joint" type="fixed">
-        <parent link="${prefix}D435_camera" />
+        <parent link="${prefix}d435_camera" />
         <child link="${prefix}ired2" />
         <origin xyz="0 0.01 0.004" rpy="0 0 0"/>
@@ -75,9 +75,9 @@
     <!-- Load plugin to the model ("robot" in urdf format)-->
     <gazebo>
-        <plugin name="${prefix}D435" filename="librealsense_gazebo_plugin.so"/>
+        <plugin name="${prefix}d435" filename="librealsense_gazebo_plugin.so"/>
         <!--<pose frame="">0 0 0.015 0 0 0</pose>-->
     </gazebo>
     <!-- Load parameters to model's main link-->
-    <gazebo reference="${prefix}D435_camera">
+    <gazebo reference="${prefix}d435_camera">
         <self_collide>0</self_collide>
         <enable_wind>0</enable_wind>
@@ -95,5 +95,5 @@
         <sensor name="color" type="camera">
             <pose frame="">0 -0.046 0.004 0 0 0</pose>
-            <camera name="${prefix}D435_camera">
+            <camera name="${prefix}d435_camera">
             <horizontal_fov>1.047</horizontal_fov>
             <image>
@@ -118,5 +118,5 @@
         <sensor name="ired1" type="camera">
             <pose frame="">0 -0.06 0.004 0 0 0</pose>
-            <camera name="${prefix}D435_camera">
+            <camera name="${prefix}d435_camera">
             <horizontal_fov>1.047</horizontal_fov>
             <image>
@@ -141,5 +141,5 @@
         <sensor name="ired2" type="camera">
             <pose frame="">0 0.01 0.004 0 0 0</pose>
-            <camera name="${prefix}D435_camera">
+            <camera name="${prefix}d435_camera">
             <horizontal_fov>1.047</horizontal_fov>
             <image>
@@ -164,5 +164,5 @@
         <sensor name="depth" type="depth">
             <pose frame="">0 -0.046 0.004 0 0 0</pose>
-            <camera name="${prefix}D435_camera">
+            <camera name="${prefix}d435_camera">
             <horizontal_fov>1.047</horizontal_fov>
             <image>

File: urdf/realsense-r200.macro.xacro (robot description, xacro)
@@ -2,5 +2,5 @@
 <!--Develped by Daniel Ordonez 22.05.2018 - daniels.ordonez@gmail.com
     INFORMATION:
-        This xacro file a URDF representation of the intel real sense RS200 with the
+        This xacro file a URDF representation of the intel real sense R200 with the
         virtual links representing the position of:
             * The RGB color camera
@@ -11,11 +11,11 @@
 -->
 <robot xmlns:xacro="http://ros.org/wiki/xacro">
-<xacro:macro name="realsense-rs200" params="prefix parent *origin">
+<xacro:macro name="realsense-r200" params="prefix parent *origin">
     <!-- Camera link -->
-    <link name="${prefix}rs200_camera">
+    <link name="${prefix}r200_camera">
         <visual>
             <origin rpy="0 0 0" xyz="0 0 0"/>
             <geometry>
-                <mesh filename="package://realsense_gazebo_plugin/models/realsense_camera/meshes/realsense.dae"/>
+                <mesh filename="package://realsense_gazebo_plugin/models/realsense_camera/meshes/realsense_r200.dae"/>
             </geometry>
         </visual>
@@ -40,5 +40,5 @@
     <joint name="${prefix}realsense_joint" type="fixed">
         <parent link="${parent}"/>
-        <child link="${prefix}rs200_camera"/>
+        <child link="${prefix}r200_camera"/>
         <xacro:insert_block name="origin"/>
     </joint>
@@ -50,5 +50,5 @@
     <!-- Joints positioning the virtual links with respect to the camera main link-->
     <joint name="${prefix}color_joint" type="fixed">
-        <parent link="${prefix}rs200_camera" />
+        <parent link="${prefix}r200_camera" />
         <child link="${prefix}color" />
         <!-- <origin xyz="0 -0.046 0.004" rpy="0 0 0"/> -->
@@ -57,15 +57,15 @@
     </joint>
     <joint name="${prefix}depth_joint" type="fixed">
-        <parent link="${prefix}rs200_camera" />
+        <parent link="${prefix}r200_camera" />
         <child link="${prefix}depth" />
         <origin xyz="0 -0.03 0.004" rpy="0 0 0"/>
     </joint>
     <joint name="${prefix}ired1_joint" type="fixed">
-        <parent link="${prefix}rs200_camera" />
+        <parent link="${prefix}r200_camera" />
         <child link="${prefix}ired1" />
         <origin xyz="0 -0.06 0.004" rpy="0 0 0"/>
     </joint>
     <joint name="${prefix}ired2_joint" type="fixed">
-        <parent link="${prefix}rs200_camera" />
+        <parent link="${prefix}r200_camera" />
         <child link="${prefix}ired2" />
         <origin xyz="0 0.01 0.004" rpy="0 0 0"/>
@@ -79,5 +79,5 @@
     </gazebo>
     <!-- Load parameters to model's main link-->
-    <gazebo reference="${prefix}rs200_camera">
+    <gazebo reference="${prefix}r200_camera">
         <self_collide>0</self_collide>
         <enable_wind>0</enable_wind>
@@ -95,5 +95,5 @@
         <sensor name="color" type="camera">
             <pose frame="">0 -0.046 0.004 0 0 0</pose>
-            <camera name="${prefix}rs200_camera">
+            <camera name="${prefix}r200_camera">
             <horizontal_fov>1.047</horizontal_fov>
             <image>
@@ -118,5 +118,5 @@
         <sensor name="ired1" type="camera">
             <pose frame="">0 -0.06 0.004 0 0 0</pose>
-            <camera name="${prefix}rs200_camera">
+            <camera name="${prefix}r200_camera">
             <horizontal_fov>1.047</horizontal_fov>
             <image>
@@ -141,5 +141,5 @@
         <sensor name="ired2" type="camera">
             <pose frame="">0 0.01 0.004 0 0 0</pose>
-            <camera name="${prefix}rs200_camera">
+            <camera name="${prefix}r200_camera">
             <horizontal_fov>1.047</horizontal_fov>
             <image>
@@ -164,5 +164,5 @@
         <sensor name="depth" type="depth">
             <pose frame="">0 -0.046 0.004 0 0 0</pose>
-            <camera name="${prefix}rs200_camera">
+            <camera name="${prefix}r200_camera">
             <horizontal_fov>1.047</horizontal_fov>
             <image>
